File: 379-382-Arduino-DIY-KiCAD/zArduino/zArduino.kicad_pcb (KiCad board)
At the start: 2 copper layers, 68.8 x 53.6 mm, 46 parts, among them J1 USB_B, J2 Barrel_Jack_Switch, J3 Conn_01x04_Female, J4 Conn_01x06_Female, J5 Conn_01x06_Female, J6 Conn_02x03_Odd_Even, J7 Conn_01x08_Female, J8 Conn_01x08_Female, J9 Conn_01x02_Female, Q1 NDT2955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

Commit message: karzuino?
Other:
- net class Default removed
